File: Eagle Files/Projects/Revised Block Diagram/Detailed Block Diagram.sch (EAGLE design)
At the start: 19 parts

Commit message: Eagle Schematic Updated
Parts:
- removed FUSE: 800A, Custom Block Diagram Parts:FUSE
- added AIR1, AIR2, AIR3, AIR4: AIR, Custom Block Diagram Parts:AIR
- added FUSE1, FUSE2, FUSE3, FUSE4: FUSE, Custom Block Diagram Parts:FUSE
- added HVD1, HVD2, HVD3, HVD4: HVD, Custom Block Diagram Parts:HVD
- added R1, R2, R3, R4, R5, R6, R7, R8: (no value), resistor:R-US_0817/22
- added U$19, U$20, U$21, U$22, U$23, U$24, U$25, U$26, U$27, U$28, U$29, U$30, U$31, U$32, U$33, U$34, U$35, U$36, U$37, U$38, U$39, U$40, U$41, U$42, U$43, U$44, U$45, U$46, U$47, U$48, U$49, U$50, U$51, U$52, U$53, U$54, U$55, U$56, U$57, U$58, U$59, U$60, U$61, U$62, U$63, U$64, U$65, U$66, U$67, U$68, U$69, U$70, U$71, U$72, U$73, U$74, U$75, U$76, U$77, U$78, U$79, U$80, U$81, U$82, U$83, U$84: BAT_CELL, Custom Block Diagram Parts:BAT_CELL
Connections:
- new net B$1: R1.1, R2.1, R3.1, R4.1, R5.1, R6.1, R7.1, R8.1, U$1.+, U$10.+, U$11.+, U$12.+, U$13.+, U$14.+, U$15.+, U$16.+, U$17.+, U$18.+, U$19.+, U$2.+, U$20.+, U$21.+, U$22.+, U$23.+, U$24.+, U$25.+, U$26.+, U$27.+, U$28.+, U$29.+, U$3.+, U$30.+, U$31.+, U$32.+, U$33.+, U$34.+, U$35.+, U$36.+, U$37.+, U$38.+, U$39.+, U$4.+, U$40.+, U$41.+, U$42.+, U$43.+, U$44.+, U$45.+, U$46.+, U$47.+, U$48.+, U$49.+, U$5.+, U$50.+, U$51.+, U$52.+, U$53.+, U$54.+, U$55.+, U$56.+, U$57.+, U$58.+, U$59.+, U$60.+, U$61.+, U$62.+, U$63.+, U$64.+, U$65.+, U$66.+, U$67.+, U$68.+, U$73.+, U$74.+, U$75.+, U$76.+, U$77.+, U$78.+, U$79.+, U$80.+, U$81.+, U$82.+, U$83.+, U$84.+
- new net N$1: R1.2, U$9.+
- new net N$2: R2.2, U$8.+
- new net N$3: R3.2, U$7.+
- new net N$4: R4.2, U$6.+
- new net N$5: R5.2, U$72.+
- new net N$6: R6.2, U$71.+
- new net N$7: R7.2, U$70.+
- new net N$8: R8.2, U$69.+
Other:
- note added: "...One for every battery"
- note added: "Orion BMS"
- note added: "TSV (+)"
- note added: "TSV (-)"
- note added: "Therm Expansion"
